File: main_board/irrigation_ctrl_main_board.kicad_pcb (KiCad board)
At the start: 2 copper layers, 120 x 72.4 mm, 84 parts, among them J1 UART1, J10 Conn_01x01, J11 Conn_01x01, J12 Conn_01x01, J13 Conn_01x01, J2 UART2, J3 JTAG, J4 VSPI, J5 UART_DBG, J6 PWR_IN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

Commit message: Preparations for publication
Parts:
- added REF***: OSHW-Logo_5.7x6mm_SilkScreen, Symbols:OSHW-Logo_5.7x6mm_SilkScreen, F.Cu at (124.5, 174.0)
- moved Q3 0.19 mm to (78.7, 169.5), turned to 90 degrees
Connections:
- Q3 pad 2: IO0 -> DTR0
- Q3 pad 3: DTR0 -> IO0
Routing:
- net RTS0: track 18.5 -> 22.0 mm
- net DTR0: track 8.75 -> 10.8 mm
- net Net-(Q3-Pad1): track 2.81 -> 4.73 mm
- net IO0: track 56.0 -> 56.6 mm
Other:
- board text added: "Irrigation Ctrl MW 12/17"
- board text added: "Licensed under BSD-3-Clause"
- board text removed: "Irrigation Ctrl MW 10/17"
